File: rails_signal_feedback_dcc-railcom-8x50_test.kicad_sch (KiCad schematic)
At the start: 5 parts, among them J201 Conn_02x05_Odd_Even

Commit message: Fix - Test für RC 8x50
Parts:
- renumbered R202 to R201, R201 to R202
Connections:
- net +3V3: now also J201.4 (Pin_4); no longer J201.2 (Pin_2)
- net +J_3v3: now also J201.3 (Pin_3); no longer J201.1 (Pin_1)
- net J_RAILCOM_DATA: now also J201.1 (Pin_1); no longer J201.3 (Pin_3)
- net RAILCOM_DATA: now also J201.2 (Pin_2); no longer J201.4 (Pin_4)
- no-connect marks 1 -> 5
Other:
- sheet rails_signal_feedback_dcc-railcom-8x50 ports: added none; removed _TST_RC_CURR, _TST_RC_DATA_IN, _TST_RC_J_SIGNAL, _TST_RC_ON_OFF, _TST_RC_SIGNAL
