File: rails_power_ac-dc-bridge-medium-3xs-test.kicad_sch (KiCad schematic)
At the start: 1 part, among them J101 Conn_02x04_Odd_Even

Commit message: Fix - Ac-Dc Bridge Medium test
Connections:
- net +U is gone; now on net U+: J101.1 (Pin_1)
- no-connect marks 0 -> 4
Changed lines of the file:
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@@
 		(company "Chatelain Engineering, Bern - CH")
+	)
+	(no_connect
+		(at 24.13 60.96)
+	)
+	(no_connect
+		(at 24.13 63.5)
+	)
+	(no_connect
+		(at 24.13 58.42)
+	)
+	(no_connect
+		(at 24.13 55.88)
 	)
 	(bus
@@
 	(label "J_AC[0..1]"
 		(at 116.84 55.88 180)
-		(fields_autoplaced yes)
 		(effects
 			(font
@@
 	(label "J_U"
 		(at 90.17 35.56 180)
-		(fields_autoplaced yes)
 		(effects
 			(font
@@
 	(label "J_AC1"
 		(at 59.69 63.5 180)
-		(fields_autoplaced yes)
-		(effects
-			(font
-				(size 1.27 1.27)
-			)
-			(justify right bottom)
-		)
-	)
-	(label "+U"
+		(effects
+			(font
+				(size 1.27 1.27)
+			)
+			(justify right bottom)
+		)
+	)
+	(label "U+"
 		(at 24.13 55.88 0)
-		(fields_autoplaced yes)
 		(effects
 			(font
@@
 	(label "AC1"
 		(at 24.13 63.5 0)
-		(fields_autoplaced yes)
 		(effects
 			(font
@@
 	(label "AC0"
 		(at 24.13 60.96 0)
-		(fields_autoplaced yes)
 		(effects
 			(font
@@
 	(label "J_GND"
 		(at 59.69 58.42 180)
-		(fields_autoplaced yes)
 		(effects
 			(font
@@
 	(label "GND"
 		(at 24.13 58.42 0)
-		(fields_autoplaced yes)
 		(effects
 			(font
@@
 	(label "J_AC0"
 		(at 59.69 60.96 180)
-		(fields_autoplaced yes)
 		(effects
 			(font
@@
 	(label "J_GND"
 		(at 88.9 78.74 180)
-		(fields_autoplaced yes)
 		(effects
 			(font
@@
 	(label "J_U"
 		(at 59.69 55.88 180)
-		(fields_autoplaced yes)
 		(effects
 			(font
@@
 	(hierarchical_label "GND"
 		(shape output)
-		(at 41.91 38.1 0)
-		(fields_autoplaced yes)
-		(effects
-			(font
-				(size 1.27 1.27)
-			)
-			(justify left)
+		(at 24.13 58.42 180)
+		(effects
+			(font
+				(size 1.27 1.27)
+			)
+			(justify right)
 		)
 	)
 	(hierarchical_label "U+"
 		(shape output)
-		(at 41.91 35.56 0)
-		(fields_autoplaced yes)
-		(effects
-			(font
-				(size 1.27 1.27)
-			)
-			(justify left)
+		(at 24.13 55.88 180)
+		(effects
+			(font
+				(size 1.27 1.27)
+			)
+			(justify right)
 		)
 	)
@@
 		(shape input)
 		(at 33.02 35.56 180)
-		(fields_autoplaced yes)
-		(effects
-			(font
+		(effects
+			(font
